File: opk-pi-1wire-i2c-v1.brd (EAGLE design)
At the start: 33.8 x 52.6 mm, 12 parts, among them U1 RJ45, U2 RJ11

Commit message: update
Connections:
- removed net 23: R1.1
- net 4: now also R1.1
Routing:
- net 4: track 0.00 -> 145.8 mm
- net 3V3: track 0.00 -> 143.9 mm
- net GND: track 0.00 -> 141.8 mm
- net 15-RX: track 0.00 -> 31.9 mm
- net 14-TX: track 0.00 -> 31.3 mm
- net 5V: track 0.00 -> 29.9 mm
- net 3-SCL: track 0.00 -> 23.3 mm
- net 2-SDA: track 0.00 -> 21.7 mm
