File: opk-pi-1wire-i2c-v1.brd (EAGLE design)
At the start: 33.8 x 52.6 mm, 12 parts, among them U1 RJ45, U2 RJ11

Commit message: update
Parts:
- moved SV1 0.55 mm to (16.8, 26.5)
Connections:
- net 4: now also JP5.1, JP6.1, JP7.1; no longer JP5.3, JP6.3, JP7.3
- net GND: now also JP5.3, JP6.3, JP7.3; no longer JP5.1, JP6.1, JP7.1
Routing:
- net 5V: track 29.9 -> 48.7 mm
- net GND: track 141.8 -> 134.5 mm
- net 3V3: track 143.9 -> 140.6 mm
- net 4: track 145.8 -> 143.0 mm
- net 15-RX: track 31.9 -> 33.8 mm
- net 2-SDA: track 21.7 -> 22.3 mm
- net 3-SCL: track 23.3 -> 23.8 mm
Other:
- board text added: "RJ11"
- board text added: "RJ45"
